Commit message: Remove 'world' joint from panda_arm macro

File: franka_description/robots/panda_arm.xacro (robot description, xacro)
@@ -10,10 +10,4 @@
     </xacro:unless>
     <!-- for simulation -->
-    <link name="world" />
-    <joint name="robot_to_world" type="fixed">
-      <parent link="world" />
-      <child link="${arm_id}_link0" />
-      <origin xyz="0.0 0.0 0.0" rpy="0.0 0.0 0.0" />
-    </joint>
     <xacro:property name="joint_damping" value="1.0"/>
     <!-- end for simulation -->
